Commit message: Edited transmission to position control interface

File: ur_description/urdf/ur10.transmission.xacro (robot description, xacro)
@@ -1,53 +1,65 @@
 <?xml version="1.0"?>
 <robot xmlns:xacro="http://www.ros.org/wiki/xacro">
-  <xacro:macro name="ur10_arm_transmission" params="prefix">
-    <transmission name="${prefix}shoulder_pan_trans">
-      <type>transmission_interface/SimpleTransmission</type>
-      <joint name="${prefix}shoulder_pan_joint"/>
-      <actuator name="${prefix}shoulder_pan_motor">
-        <hardwareInterface>EffortJointInterface</hardwareInterface>
-        <mechanicalReduction>1</mechanicalReduction>
-      </actuator>
-    </transmission>
-    <transmission name="${prefix}shoulder_lift_trans">
-      <type>transmission_interface/SimpleTransmission</type>
-      <joint name="${prefix}shoulder_lift_joint"/>
-      <actuator name="${prefix}shoulder_lift_motor">
-        <hardwareInterface>EffortJointInterface</hardwareInterface>
-        <mechanicalReduction>1</mechanicalReduction>
-      </actuator>
-    </transmission>
-    <transmission name="${prefix}elbow_trans">
-      <type>transmission_interface/SimpleTransmission</type>
-      <joint name="${prefix}elbow_joint"/>
-      <actuator name="${prefix}elbow_motor">
-        <hardwareInterface>EffortJointInterface</hardwareInterface>
-        <mechanicalReduction>1</mechanicalReduction>
-      </actuator>
-    </transmission>
-    <transmission name="${prefix}wrist_1_trans">
-      <type>transmission_interface/SimpleTransmission</type>
-      <joint name="${prefix}wrist_1_joint"/>
-      <actuator name="${prefix}wrist_1_motor">
-        <hardwareInterface>EffortJointInterface</hardwareInterface>
-        <mechanicalReduction>1</mechanicalReduction>
-      </actuator>
-    </transmission>
-    <transmission name="${prefix}wrist_2_trans">
-      <type>transmission_interface/SimpleTransmission</type>
-      <joint name="${prefix}wrist_2_joint"/>
-      <actuator name="${prefix}wrist_2_motor">
-        <hardwareInterface>EffortJointInterface</hardwareInterface>
-        <mechanicalReduction>1</mechanicalReduction>
-      </actuator>
-    </transmission>
-    <transmission name="${prefix}wrist_3_trans">
-      <type>transmission_interface/SimpleTransmission</type>
-      <joint name="${prefix}wrist_3_joint"/>
-      <actuator name="${prefix}wrist_3_motor">
-        <hardwareInterface>EffortJointInterface</hardwareInterface>
-        <mechanicalReduction>1</mechanicalReduction>
-      </actuator>
-    </transmission>
-  </xacro:macro>
+    <xacro:macro name="ur10_arm_transmission" params="prefix">
+        <transmission name="${prefix}shoulder_pan_trans">
+            <type>transmission_interface/SimpleTransmission</type>
+            <joint name="${prefix}shoulder_pan_joint">
+                <hardwareInterface>PositionJointInterface</hardwareInterface>
+            </joint>
+            <actuator name="${prefix}shoulder_pan_motor">
+                <hardwareInterface>PositionJointInterface</hardwareInterface>
+                <mechanicalReduction>1</mechanicalReduction>
+            </actuator>
+        </transmission>
+        <transmission name="${prefix}shoulder_lift_trans">
+            <type>transmission_interface/SimpleTransmission</type>
+            <joint name="${prefix}shoulder_lift_joint">
+                <hardwareInterface>PositionJointInterface</hardwareInterface>
+            </joint>
+            <actuator name="${prefix}shoulder_lift_motor">
+                <hardwareInterface>PositionJointInterface</hardwareInterface>
+                <mechanicalReduction>1</mechanicalReduction>
+            </actuator>
+        </transmission>
+        <transmission name="${prefix}elbow_trans">
+            <type>transmission_interface/SimpleTransmission</type>
+            <joint name="${prefix}elbow_joint">
+                <hardwareInterface>PositionJointInterface</hardwareInterface>
+            </joint>
+            <actuator name="${prefix}elbow_motor">
+                <hardwareInterface>PositionJointInterface</hardwareInterface>
+                <mechanicalReduction>1</mechanicalReduction>
+            </actuator>
+        </transmission>
+        <transmission name="${prefix}wrist_1_trans">
+            <type>transmission_interface/SimpleTransmission</type>
+            <joint name="${prefix}wrist_1_joint">
+                <hardwareInterface>PositionJointInterface</hardwareInterface>
+            </joint>
+            <actuator name="${prefix}wrist_1_motor">
+                <hardwareInterface>PositionJointInterface</hardwareInterface>
+                <mechanicalReduction>1</mechanicalReduction>
+            </actuator>
+        </transmission>
+        <transmission name="${prefix}wrist_2_trans">
+            <type>transmission_interface/SimpleTransmission</type>
+            <joint name="${prefix}wrist_2_joint">
+                <hardwareInterface>PositionJointInterface</hardwareInterface>
+            </joint>
+            <actuator name="${prefix}wrist_2_motor">
+                <hardwareInterface>PositionJointInterface</hardwareInterface>
+                <mechanicalReduction>1</mechanicalReduction>
+            </actuator>
+        </transmission>
+        <transmission name="${prefix}wrist_3_trans">
+            <type>transmission_interface/SimpleTransmission</type>
+            <joint name="${prefix}wrist_3_joint">
+                <hardwareInterface>PositionJointInterface</hardwareInterface>
+            </joint>
+            <actuator name="${prefix}wrist_3_motor">
+                <hardwareInterface>PositionJointInterface</hardwareInterface>
+                <mechanicalReduction>1</mechanicalReduction>
+            </actuator>
+        </transmission>
+    </xacro:macro>
 </robot>

File: ur_description/urdf/ur5.transmission.xacro (robot description, xacro)
@@ -4,7 +4,9 @@
     <transmission name="${prefix}shoulder_pan_trans">
       <type>transmission_interface/SimpleTransmission</type>
-      <joint name="${prefix}shoulder_pan_joint"/>
+      <joint name="${prefix}shoulder_pan_joint">
+        <hardwareInterface>PositionJointInterface</hardwareInterface>
+      </joint>
       <actuator name="${prefix}shoulder_pan_motor">
-        <hardwareInterface>EffortJointInterface</hardwareInterface>
+        <hardwareInterface>PositionJointInterface</hardwareInterface>
         <mechanicalReduction>1</mechanicalReduction>
       </actuator>
@@ -12,7 +14,9 @@
     <transmission name="${prefix}shoulder_lift_trans">
       <type>transmission_interface/SimpleTransmission</type>
-      <joint name="${prefix}shoulder_lift_joint"/>
+      <joint name="${prefix}shoulder_lift_joint">
+        <hardwareInterface>PositionJointInterface</hardwareInterface>
+      </joint>
       <actuator name="${prefix}shoulder_lift_motor">
-        <hardwareInterface>EffortJointInterface</hardwareInterface>
+        <hardwareInterface>PositionJointInterface</hardwareInterface>
         <mechanicalReduction>1</mechanicalReduction>
       </actuator>
@@ -20,7 +24,9 @@
     <transmission name="${prefix}elbow_trans">
       <type>transmission_interface/SimpleTransmission</type>
-      <joint name="${prefix}elbow_joint"/>
+      <joint name="${prefix}elbow_joint">
+        <hardwareInterface>PositionJointInterface</hardwareInterface>
+      </joint>
       <actuator name="${prefix}elbow_motor">
-        <hardwareInterface>EffortJointInterface</hardwareInterface>
+        <hardwareInterface>PositionJointInterface</hardwareInterface>
         <mechanicalReduction>1</mechanicalReduction>
       </actuator>
@@ -28,7 +34,9 @@
     <transmission name="${prefix}wrist_1_trans">
       <type>transmission_interface/SimpleTransmission</type>
-      <joint name="${prefix}wrist_1_joint"/>
+      <joint name="${prefix}wrist_1_joint">
+        <hardwareInterface>PositionJointInterface</hardwareInterface>
+      </joint>
       <actuator name="${prefix}wrist_1_motor">
-        <hardwareInterface>EffortJointInterface</hardwareInterface>
+        <hardwareInterface>PositionJointInterface</hardwareInterface>
         <mechanicalReduction>1</mechanicalReduction>
       </actuator>
@@ -36,7 +44,9 @@
     <transmission name="${prefix}wrist_2_trans">
       <type>transmission_interface/SimpleTransmission</type>
-      <joint name="${prefix}wrist_2_joint"/>
+      <joint name="${prefix}wrist_2_joint">
+        <hardwareInterface>PositionJointInterface</hardwareInterface>
+      </joint>
       <actuator name="${prefix}wrist_2_motor">
-        <hardwareInterface>EffortJointInterface</hardwareInterface>
+        <hardwareInterface>PositionJointInterface</hardwareInterface>
         <mechanicalReduction>1</mechanicalReduction>
       </actuator>
@@ -44,7 +54,9 @@
     <transmission name="${prefix}wrist_3_trans">
       <type>transmission_interface/SimpleTransmission</type>
-      <joint name="${prefix}wrist_3_joint"/>
+      <joint name="${prefix}wrist_3_joint">
+        <hardwareInterface>PositionJointInterface</hardwareInterface>
+      </joint>
       <actuator name="${prefix}wrist_3_motor">
-        <hardwareInterface>EffortJointInterface</hardwareInterface>
+        <hardwareInterface>PositionJointInterface</hardwareInterface>
         <mechanicalReduction>1</mechanicalReduction>
       </actuator>
