Commit message: Arm prefix Added arm_prefix to xacros. hacked / hard coded the arm_prefix into ur_moveit_plugin.cpp as I was unable to set this parameter in yaml files. Needs to check this.

File: ur_description/urdf/ur10_joint_limited_robot.urdf.xacro (robot description, xacro)
@@ -6,10 +6,11 @@
   <!-- ur10 -->
   <xacro:include filename="$(find ur_description)/urdf/ur10.urdf.xacro" />
+  <xacro:property name="arm_prefix" value="ur10_" />
   <!-- arm -->
-  <xacro:ur10_robot prefix="" joint_limited="true"/>
+  <xacro:ur10_robot prefix="${arm_prefix}" joint_limited="true"/>
   <link name="world" />
   <joint name="world_joint" type="fixed">
     <parent link="world" />
-    <child link = "base_link" />
+    <child link = "${arm_prefix}base_link" />
     <origin xyz="0.0 0.0 0.0" rpy="0.0 0.0 0.0" />
   </joint>

File: ur_description/urdf/ur10_robot.urdf.xacro (robot description, xacro)
@@ -6,10 +6,11 @@
   <!-- ur10 -->
   <xacro:include filename="$(find ur_description)/urdf/ur10.urdf.xacro" />
+  <xacro:property  name="arm_prefix" value="ur10_" />
   <!-- arm -->
-  <xacro:ur10_robot prefix="" joint_limited="false"/>
+  <xacro:ur10_robot prefix="${arm_prefix}" joint_limited="false"/>
   <link name="world" />
   <joint name="world_joint" type="fixed">
     <parent link="world" />
-    <child link = "base_link" />
+    <child link = "${arm_prefix}base_link" />
     <origin xyz="0.0 0.0 0.0" rpy="0.0 0.0 0.0" />
   </joint>
